File: HW/KAKAPO-20A.kicad_pcb (KiCad board)
At the start: 4 copper layers, 51.5 x 28 mm, 95 parts, among them J1 Pins_2.54_1x3, J2 Pins_2.54_1x3, J3 Pins_2.54_1x3, J4 Pins_2.54_1x3, M1 Mount_M3, M2 Mount_M3, M3 Mount_M3, M4 Mount_M3, U1 DRV8244S-Q1, U2 DRV8244S-Q1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

Commit message: Update Part Numbers For Second Release
Other:
- board text added: "KAKAPO ESC v0.2"
- board text removed: "KAKAPO ESC v0.1"

Commit message: Update Switch NPTH Geometry and VBatt Circuit
Routing:
- net VCC: track 42.8 -> 39.4 mm, vias 55 -> 54
Other:
- board text added: "KAKAPO ESC v1.0"
- board text removed: "KAKAPO ESC v0.2"
Changed lines of the file:
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@@
   (title_block
     (title "KAKAPO - 20A")
-    (date "2024-04-28")
-    (rev "v0.2")
+    (date "2024-06-15")
+    (rev "v1.0")
     (company "CB-TECHNOLOGY")
   )
@@
     (fp_arc (start 1.5 -3.9) (mid 4.180396 0) (end 1.5 3.9)
       (stroke (width 1.6) (type default)) (layer "F.Paste"))
+    (fp_circle (center 0 0) (end 3.175 0)
+      (stroke (width 0.1) (type default)) (fill none) (layer "Edge.Cuts"))
     (fp_circle (center 0 0) (end 5.2 0)
       (stroke (width 0.05) (type solid)) (fill none) (layer "F.CrtYd"))
     (fp_circle (center 0 0) (end 5.2 0)
       (stroke (width 0.15) (type solid)) (fill none) (layer "F.Fab"))
-    (pad "" np_thru_hole circle (at 0 0) (size 6.35 6.35) (drill 6.35) (layers "F.Cu" "F.Mask")
-      (clearance 0.2))
-    (pad "1" smd circle (at 0 0) (size 10 10) (layers "F.Cu" "F.Mask")
+    (pad "1" smd circle (at 0 0) (size 10 10) (layers "F.Cu" "F.Paste" "F.Mask")
       (net 2 "VCC") (pinfunction "1") (pintype "passive") (clearance 0.2))
     (pad "2" smd circle (at 0 0) (size 10 10) (layers "B.Cu" "B.Mask")
@@
     )
     (stroke (width 0.2) (type solid)) (fill solid) (layer "F.Cu"))
-  (gr_rect (start 238.5 112.5) (end 243.5 128)
+  (gr_rect (start 242.19 114.19) (end 243.5 116)
+    (stroke (width 0) (type solid)) (fill solid) (layer "B.Cu"))
+  (gr_rect (start 238.5 116) (end 243.5 128)
     (stroke (width 0) (type solid)) (fill solid) (layer "B.Cu"))
   (gr_rect (start 232.5 122.4) (end 243.5 128)
@@
     (effects (font (size 0.8 0.8) (thickness 0.2) bold) (justify mirror))
   )
-  (gr_text "KAKAPO ESC v0.2" (at 209 110.5) (layer "B.SilkS")
+  (gr_text "KAKAPO ESC v1.0" (at 209 110.5) (layer "B.SilkS")
     (effects (font (size 1.2 1.2) (thickness 0.25) bold) (justify right mirror))
   )
@@
   (segment (start 232.4 106.9) (end 230.475 106.9) (width 0.2) (layer "B.Cu") (net 1))
   (segment (start 230.475 106.9) (end 228.525 104.95) (width 0.2) (layer "B.Cu") (net 1))
-  (segment (start 234.86 112.035) (end 235.325 112.5) (width 1) (layer "F.Cu") (net 2))
   (segment (start 215.5 116.9) (end 211.5 116.9) (width 0.4) (layer "F.Cu") (net 2))
   (segment (start 238.48 105.51356) (end 238.536341 105.46474) (width 0.2) (layer "F.Cu") (net 2))
   (segment (start 225.8 115.95) (end 226.1 116.25) (width 0.5) (layer "F.Cu") (net 2))
   (segment (start 225.2 115.95) (end 225.8 115.95) (width 0.5) (layer "F.Cu") (net 2))
-  (segment (start 235.184212 110.765) (end 236.224606 109.724606) (width 1) (layer "F.Cu") (net 2))
   (segment (start 238.76 119.25) (end 238.75 119.24) (width 0.2) (layer "F.Cu") (net 2))
   (segment (start 238.7 105.301081) (end 238.7 102.8) (width 0.2) (layer "F.Cu") (net 2))
   (segment (start 222.98 116.9) (end 223.5 116.9) (width 0.4) (layer "F.Cu") (net 2))
-  (segment (start 240.300762 116.325762) (end 241.563262 115.063262) (width 0.4) (layer "F.Cu") (net 2))
   (segment (start 225.2 115.95) (end 224.9 116.25) (width 0.5) (layer "F.Cu") (net 2))
   (segment (start 214.1 116.25) (end 214.1 116.9) (width 0.5) (layer "F.Cu") (net 2))
   (segment (start 224.9 116.45) (end 226.1 116.45) (width 0.5) (layer "F.Cu") (net 2))
   (segment (start 212.9 116.25) (end 212.9 116.9) (width 0.5) (layer "F.Cu") (net 2))
-  (segment (start 238.48 111.52) (end 239 111) (width 0.2) (layer "F.Cu") (net 2))
   (segment (start 215.35 116.9) (end 213.5 116.9) (width 0.4) (layer "F.Cu") (net 2))
   (segment (start 213.8 115.95) (end 214.1 116.25) (width 0.5) (layer "F.Cu") (net 2))
@@
   (segment (start 212.9 116.45) (end 214.1 116.45) (width 0.5) (layer "F.Cu") (net 2))
   (segment (start 238.48 105.521081) (end 238.48 106.2) (width 0.2) (layer "F.Cu") (net 2))
+  (segment (start 238.75 119.24) (end 238.75 118.846266) (width 0.4) (layer "F.Cu") (net 2))
   (segment (start 213.2 115.95) (end 212.9 116.25) (width 0.5) (layer "F.Cu") (net 2))
   (segment (start 238.7 102.8) (end 240.5 102.8) (width 0.2) (layer "F.Cu") (net 2))
@@
   (segment (start 226.1 116.25) (end 226.1 116.9) (width 0.5) (layer "F.Cu") (net 2))
   (segment (start 227.5 116.9) (end 223.5 116.9) (width 0.4) (layer "F.Cu") (net 2))
-  (segment (start 238.75 118.75) (end 238.75 119.24) (width 0.4) (layer "F.Cu") (net 2))
+  (segment (start 238.75 118.846266) (end 237.762769 117.859035) (width 0.4) (layer "F.Cu") (net 2))
   (segment (start 224.9 116.25) (end 224.9 116.9) (width 0.5) (layer "F.Cu") (net 2))
   (segment (start 248.05 108) (end 248.05 120) (width 0.6) (layer "F.Cu") (net 2))
@@
   (via (at 240 100.5) (size 0.5) (drill 0.3) (layers "F.Cu" "B.Cu") (net 2))
   (via (at 239 101.5) (size 0.5) (drill 0.3) (layers "F.Cu" "B.Cu") (net 2))
-  (via (at 238.75 118.75) (size 0.4) (drill 0.25) (layers "F.Cu" "B.Cu") (net 2))
   (via (at 235.391675 116.650903) (size 0.4) (drill 0.25) (layers "F.Cu" "B.Cu") (free) (net 2))
   (via (at 248.75 114) (size 0.4) (drill 0.25) (layers "F.Cu" "B.Cu") (free) (net 2))

Commit message: Fix Motor Driver Comms Tracking Issue
Parts:
- R22: value 22.1K 1% -> 22K 1%
- moved D1 0.30 mm to (202.7, 108.8)
Changed lines of the file:
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@@
         (effects (font (size 0.26 0.26) (thickness 0.04)))
     )
+    (fp_line (start -1 -0.2) (end -1 0.2)
+      (stroke (width 0.2) (type default)) (layer "F.SilkS"))
     (fp_line (start -0.153641 -0.38) (end 0.153641 -0.38)
       (stroke (width 0.15) (type solid)) (layer "F.SilkS"))
@@
   )
   (footprint "R_Resistor:R_0402" (layer "F.Cu")
-    (at 202.7 109.1 90)
+    (at 202.7 108.8 90)
     (property "LCSC Part" "C2837790")
     (property "Params" "40V,1A,600mV")
@@
         (effects (font (size 0.26 0.26) (thickness 0.04)))
     )
+    (fp_line (start -1 -0.2) (end -1 0.2)
+      (stroke (width 0.2) (type default)) (layer "F.SilkS"))
     (fp_line (start -0.153641 -0.38) (end 0.153641 -0.38)
       (stroke (width 0.15) (type solid)) (layer "F.SilkS"))
@@
         (effects (font (size 1 1) (thickness 0.15)))
     )
-    (fp_text value "22.1K 1%" (at 0 1.27) (layer "F.Fab") hide
+    (fp_text value "22K 1%" (at 0 1.27) (layer "F.Fab") hide
         (effects (font (size 1 1) (thickness 0.15)))
     )
@@
   )
   (segment (start 206.5 107.2) (end 203.3 107.2) (width 0.5) (layer "F.Cu") (net 1))
-  (segment (start 203.3 107.2) (end 202.7 107.8) (width 0.5) (layer "F.Cu") (net 1))
+  (segment (start 202.7 107.8) (end 202.7 108.29) (width 0.5) (layer "F.Cu") (net 1))
   (segment (start 211.04 105.2) (end 209.3 105.2) (width 0.5) (layer "F.Cu") (net 1))
-  (segment (start 208.5 105.2) (end 206.5 107.2) (width 0.5) (layer "F.Cu") (net 1))
-  (segment (start 202.7 107.8) (end 202.7 108.59) (width 0.5) (layer "F.Cu") (net 1))
   (segment (start 232.4 106.4) (end 232.4 107.37) (width 0.4) (layer "F.Cu") (net 1))
   (segment (start 228.525 101.44) (end 228.525 105.65) (width 0.6) (layer "F.Cu") (net 1))
-  (segment (start 209.3 105.2) (end 208.5 105.2) (width 0.5) (layer "F.Cu") (net 1))
   (segment (start 209.23 108) (end 209.23 105.27) (width 0.4) (layer "F.Cu") (net 1))
+  (segment (start 203.3 107.2) (end 202.7 107.8) (width 0.5) (layer "F.Cu") (net 1))
   (segment (start 211.04 102) (end 211.04 105.2) (width 0.5) (layer "F.Cu") (net 1))
   (segment (start 209.23 105.27) (end 209.3 105.2) (width 0.2) (layer "F.Cu") (net 1))
   (segment (start 232.41 107.37) (end 232.38 107.4) (width 0.2) (layer "F.Cu") (net 1))
+  (segment (start 208.5 105.2) (end 206.5 107.2) (width 0.5) (layer "F.Cu") (net 1))
+  (segment (start 209.3 105.2) (end 208.5 105.2) (width 0.5) (layer "F.Cu") (net 1))
   (via (at 228.525 104.95) (size 0.4) (drill 0.25) (layers "F.Cu" "B.Cu") (net 1))
   (via (at 232.4 106.9) (size 0.4) (drill 0.25) (layers "F.Cu" "B.Cu") (net 1))
@@
   (segment (start 223.777207 114.15) (end 225.2 114.15) (width 0.2) (layer "B.Cu") (net 18))
   (segment (start 214.148529 113.6) (end 215.498529 114.95) (width 0.2) (layer "B.Cu") (net 18))
-  (segment (start 215.498529 114.95) (end 222.977207 114.95) (width 0.2) (layer "B.Cu") (net 18))
   (segment (start 222.977207 114.95) (end 223.777207 114.15) (width 0.2) (layer "B.Cu") (net 18))
+  (segment (start 219.9 114.95) (end 222.977207 114.95) (width 0.2) (layer "B.Cu") (net 18))
+  (segment (start 219.9 114.450001) (end 219.9 114.95) (width 0.2) (layer "B.Cu") (net 18))
+  (segment (start 215.498529 114.95) (end 219.9 114.95) (width 0.2) (layer "B.Cu") (net 18))
   (segment (start 213.2 114.042893) (end 213.642893 113.6) (width 0.2) (layer "B.Cu") (net 18))
   (segment (start 213.642893 113.6) (end 214.148529 113.6) (width 0.2) (layer "B.Cu") (net 18))
@@
   (segment (start 233.957107 118.75) (end 233.457107 118.25) (width 0.2) (layer "B.Cu") (net 28))
   (segment (start 233.25 120.26) (end 232.25 120.26) (width 0.2) (layer "F.Cu") (net 29))
-  (segment (start 202.7 109.61) (end 201.565 109.61) (width 0.5) (layer "F.Cu") (net 30))
-  (segment (start 202.7 109.61) (end 202.7 110.7) (width 0.5) (layer "F.Cu") (net 30))
   (segment (start 201.565 109.61) (end 201.5 109.675) (width 0.4) (layer "F.Cu") (net 30))
   (segment (start 202.7 113.471734) (end 202.18 113.991734) (width 0.5) (layer "F.Cu") (net 30))
+  (segment (start 202.7 109.31) (end 202.7 110.7) (width 0.5) (layer "F.Cu") (net 30))
+  (segment (start 201.565 109.61) (end 202.69 109.61) (width 0.5) (layer "F.Cu") (net 30))
   (segment (start 202.18 113.991734) (end 202.18 114.1) (width 0.5) (layer "F.Cu") (net 30))
   (segment (start 202.7 110.7) (end 202.7 113.471734) (width 0.5) (layer "F.Cu") (net 30))
+  (segment (start 202.69 109.61) (end 202.7 109.62) (width 0.5) (layer "F.Cu") (net 30))
   (segment (start 213.998924 110.7) (end 210.671076 110.7) (width 0.2) (layer "F.Cu") (net 31))
   (segment (start 209.81 114.43) (end 209.24 115) (width 0.2) (layer "F.Cu") (net 31))

Commit message: Update LED to Visible Wavelength
Parts:
- R21: value 115.8K 1% -> 118K 1%
Changed lines of the file:
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@@
   (footprint "R_Resistor:R_0402" (layer "F.Cu")
     (at 231.9 106.4 180)
-    (property "LCSC Part" "C3013150")
+    (property "LCSC Part" "")
     (property "Sheetfile" "PowerSupplies.kicad_sch")
     (property "Sheetname" "PowerSupplies")
@@
         (effects (font (size 1 1) (thickness 0.15)))
     )
-    (fp_text value "115.8K 1%" (at 0 1.27) (layer "F.Fab") hide
+    (fp_text value "118K 1%" (at 0 1.27) (layer "F.Fab") hide
         (effects (font (size 1 1) (thickness 0.15)))
     )
@@
   (footprint "R_Resistor:R_0402" (layer "F.Cu")
     (at 231.9 108.4)
-    (property "LCSC Part" "C226367")
+    (property "LCSC Part" "")
     (property "Sheetfile" "PowerSupplies.kicad_sch")
     (property "Sheetname" "PowerSupplies")
@@
     (descr "Infrared (IR) Emitter 940nm 1.2V 65mA 1mW/sr @ 20mA 20° 1206 (3216 Metric)")
     (tags "LED ReverseMount Reverse")
-    (property "LCSC Part" "C73929")
-    (property "MFG Part" "IR26-21C/L110/TR8")
+    (property "LCSC Part" "C125107")
+    (property "MFG Part" "LTST-C230KRKT")
     (property "Sheetfile" "KAKAPO-20A.kicad_sch")
     (property "Sheetname" "")

Commit message: Create v1.0 Fixed From v0.2 HW
Parts:
- moved M1 0.50 mm to (203.5, 103.0)
- moved M2 0.50 mm to (248.0, 103.0)
- moved M3 0.50 mm to (203.5, 125.0)
- moved M4 0.50 mm to (248.0, 125.0)
Connections:
- J4 pad 2: +3V3 -> +5V
Routing:
- net +3V3: track 36.3 -> 51.9 mm
- net +5V: track 25.8 -> 36.2 mm
- net GND: track 292.9 -> 282.9 mm, vias 163 -> 162
- net VCC: track 39.4 -> 34.0 mm
- net MOTOR_A-: track 5.19 -> 0.00 mm
- net MOTOR_B-: track 4.14 -> 0.00 mm
- net MOTOR_B+: track 4.14 -> 0.00 mm
- net MOTOR_A+: track 4.14 -> 0.00 mm
