File: HW/KAKAPO-20A.kicad_sch (KiCad schematic)
At the start: 50 parts, among them J1 Pins_2.54_1x3, J2 Pins_2.54_1x3, M1 Mount_M3, M2 Mount_M3, M3 Mount_M3, M4 Mount_M3

Commit message: Finish Tracking and Release For MFG
Parts:
- removed A1: Radio_FS2A, A_Assembly:Radio_FS2A, symbol A_Assembly:Radio_FS2A
- removed C11, C12: 220uF, 35V, C_Capacitor:C_6.3mm_SMD, symbol C_Capacitor:C_6.3mm_SMD
- removed R13, R14, R15, R6: 1K 1%, R_Resistor:R_0402, symbol R_Resistor:R_0402
- removed R16, R7, R8, R9: 10K 1%, R_Resistor:R_0402, symbol R_Resistor:R_0402
- added C11, C12, C15, C17, C21, C32: 22uF, 35V, C_Capacitor:C_0805, symbol C_Capacitor:C_0805
- added J3, J4: Pins_2.54_1x3, J_Connector:Pins-2.54-1x3, symbol J_Connector:Pins_2.54_1x3
- added L2, L3, L4, L5: 600R, L_Inductor:FB_0402, symbol L_Inductor:FB_0402
- DS2: LCSC Part (none) -> C73929; LCSC_Part C73929 -> (none); MFG Part (none) -> IR26-21C/L110/TR8; MFG_Part IR26-21C/L110/TR8 -> (none)
- J1, J2: LCSC Part (none) -> C429954
- S1: LCSC_Part C2916375 -> C2916373; MFG_Part SMTSO4030MTJ -> SMTSO4020MTJ
Connections:
- net +3V3: now also J4.2
- net GND: now also C11.2, C12.2, C15.2, C17.2, C21.2, C32.2, J4.3
- net RADIO_CH1: now also L2.2
- net RADIO_CH2: now also L3.2
- net RADIO_CH3: now also L4.2
- net RADIO_CH4: now also L5.2
- net VCC: now also C11.1, C12.1, C15.1, C17.1, C21.1, C32.1
- new net: J3.2, L3.1
- new net: J3.3, L4.1
- new net: J4.1, L5.1
- new net: J3.1, L2.1
Other:
- note added: "INPUT: VOLTAGE DET"
- note added: "OUTPUT: LED"
- title: KAKAPO ESC - 20A -> KAKAPO - 20A
- moved on the sheet: C23, C3, D2, DS1, DS2, DS3, R10, R11, R12, R19, R20, R24

Commit message: Update Part Numbers For Second Release
Parts:
- C11, C12, C15, C17, C21, C32: LCSC Part (none) -> C22367832; LCSC_Part C22367832 -> (none); MFG Part (none) -> HGC0805R5226M350NSLJ
- L2, L3, L4, L5: MFG Part (none) -> CBG100505U601T
- R10, R24: LCSC Part (none) -> C2077696; LCSC_Part C2077696 -> (none); MFG Part (none) -> CRCW06032K20JNEAHP; MFG_Part CRCW06032K20JNEAHP -> (none)
- S1: LCSC Part (none) -> C2916373; LCSC_Part C2916373 -> (none); MFG Part (none) -> SMTSO4020MTJ; MFG_Part SMTSO4020MTJ -> (none)
Changed lines of the file:
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@@
   (title_block
     (title "KAKAPO - 20A")
-    (date "2024-04-27")
-    (rev "v0.1")
+    (date "2024-04-28")
+    (rev "v0.2")
     (company "CB-TECHNOLOGY")
   )
@@
       (effects (font (size 0.635 0.635)) (justify left))
     )
-    (property "LCSC_Part" "C22367832" (at 87.63 41.91 0)
+    (property "LCSC Part" "C22367832" (at 87.63 41.91 0)
+      (effects (font (size 1.27 1.27)) hide)
+    )
+    (property "MFG Part" "HGC0805R5226M350NSLJ" (at 87.63 41.91 0)
       (effects (font (size 1.27 1.27)) hide)
     )
@@
       (effects (font (size 1.27 1.27)) hide)
     )
+    (property "MFG Part" "CBG100505U601T" (at 62.23 77.47 90)
+      (effects (font (size 1.27 1.27)) hide)
+    )
     (pin "1")
     (pin "2")
@@
       (effects (font (size 0.635 0.635)) (justify left))
     )
-    (property "LCSC_Part" "C22367832" (at 102.235 41.91 0)
+    (property "LCSC Part" "C22367832" (at 102.235 41.91 0)
+      (effects (font (size 1.27 1.27)) hide)
+    )
+    (property "MFG Part" "HGC0805R5226M350NSLJ" (at 102.235 41.91 0)
       (effects (font (size 1.27 1.27)) hide)
     )
@@
       (effects (font (size 1.27 1.27)) hide)
     )
+    (property "MFG Part" "CBG100505U601T" (at 62.23 90.17 90)
+      (effects (font (size 1.27 1.27)) hide)
+    )
     (pin "1")
     (pin "2")
@@
       (effects (font (size 1.27 1.27)) hide)
     )
-    (property "LCSC_Part" "C2916373" (at 58.42 48.26 0)
+    (property "LCSC Part" "C2916373" (at 58.42 48.26 0)
       (effects (font (size 1.27 1.27)) hide)
     )
-    (property "MFG_Part" "SMTSO4020MTJ" (at 58.42 50.8 0)
+    (property "MFG Part" "SMTSO4020MTJ" (at 58.42 50.8 0)
       (effects (font (size 1.27 1.27)) hide)
     )
@@
       (effects (font (size 0.635 0.635)) (justify left))
     )
-    (property "LCSC_Part" "C2077696" (at 247.015 134.62 0)
+    (property "LCSC Part" "C2077696" (at 247.015 134.62 0)
       (effects (font (size 1.27 1.27)) hide)
     )
-    (property "MFG_Part" "CRCW06032K20JNEAHP" (at 247.015 134.62 0)
+    (property "MFG Part" "CRCW06032K20JNEAHP" (at 247.015 134.62 0)
       (effects (font (size 1.27 1.27)) hide)
     )
@@
       (effects (font (size 0.635 0.635)) (justify left))
     )
-    (property "LCSC_Part" "C22367832" (at 116.84 41.91 0)
+    (property "LCSC Part" "C22367832" (at 116.84 41.91 0)
+      (effects (font (size 1.27 1.27)) hide)
+    )
+    (property "MFG Part" "HGC0805R5226M350NSLJ" (at 116.84 41.91 0)
       (effects (font (size 1.27 1.27)) hide)
     )
@@
       (effects (font (size 0.635 0.635)) (justify left))
     )
-    (property "LCSC_Part" "C22367832" (at 146.685 41.91 0)
+    (property "LCSC Part" "C22367832" (at 146.685 41.91 0)
+      (effects (font (size 1.27 1.27)) hide)
+    )
+    (property "MFG Part" "HGC0805R5226M350NSLJ" (at 146.685 41.91 0)
       (effects (font (size 1.27 1.27)) hide)
     )
@@
       (effects (font (size 0.635 0.635)) (justify left))
     )
-    (property "LCSC_Part" "C22367832" (at 72.39 41.91 0)
+    (property "LCSC Part" "C22367832" (at 72.39 41.91 0)
+      (effects (font (size 1.27 1.27)) hide)
+    )
+    (property "MFG Part" "HGC0805R5226M350NSLJ" (at 72.39 41.91 0)
       (effects (font (size 1.27 1.27)) hide)
     )
@@
       (effects (font (size 0.635 0.635)) (justify left))
     )
-    (property "LCSC_Part" "C22367832" (at 131.445 41.91 0)
+    (property "LCSC Part" "C22367832" (at 131.445 41.91 0)
+      (effects (font (size 1.27 1.27)) hide)
+    )
+    (property "MFG Part" "HGC0805R5226M350NSLJ" (at 131.445 41.91 0)
       (effects (font (size 1.27 1.27)) hide)
     )
@@
       (effects (font (size 1.27 1.27)) hide)
     )
+    (property "MFG Part" "CBG100505U601T" (at 62.23 64.77 90)
+      (effects (font (size 1.27 1.27)) hide)
+    )
     (pin "1")
     (pin "2")
@@
       (effects (font (size 1.27 1.27)) hide)
     )
+    (property "MFG Part" "CBG100505U601T" (at 62.23 102.87 90)
+      (effects (font (size 1.27 1.27)) hide)
+    )
     (pin "1")
     (pin "2")
@@
       (effects (font (size 0.635 0.635)) (justify left))
     )
-    (property "LCSC_Part" "C2077696" (at 234.95 134.62 0)
+    (property "LCSC Part" "C2077696" (at 234.95 134.62 0)
       (effects (font (size 1.27 1.27)) hide)
     )
-    (property "MFG_Part" "CRCW06032K20JNEAHP" (at 234.95 134.62 0)
+    (property "MFG Part" "CRCW06032K20JNEAHP" (at 234.95 134.62 0)
       (effects (font (size 1.27 1.27)) hide)
     )

Commit message: Update LED to Visible Wavelength
Parts:
- DS2: LCSC Part C73929 -> C125107; MFG Part IR26-21C/L110/TR8 -> LTST-C230KRKT
Changed lines of the file:
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@@
       (effects (font (size 1.27 1.27)) hide)
     )
-    (property "Datasheet" "https://www.lcsc.com/datasheet/lcsc_datasheet_1810261032_Everlight-Elec-IR26-21C-L110-TR8_C73929.pdf" (at 241.3 144.78 0)
+    (property "Datasheet" "https://www.lcsc.com/datasheet/lcsc_datasheet_1811100910_Lite-On-LTST-C230KRKT_C125107.pdf" (at 241.3 144.78 0)
       (effects (font (size 1.27 1.27)) hide)
     )
@@
       (effects (font (size 0.635 0.635)) (justify right))
     )
-    (property "LCSC Part" "C73929" (at 234.95 144.78 90)
+    (property "LCSC Part" "C125107" (at 234.95 144.78 90)
       (effects (font (size 1.27 1.27)) hide)
     )
-    (property "MFG Part" "IR26-21C/L110/TR8" (at 234.95 144.78 90)
+    (property "MFG Part" "LTST-C230KRKT" (at 234.95 144.78 90)
       (effects (font (size 1.27 1.27)) hide)
     )

Commit message: Create v1.0 Fixed From v0.2 HW
Connections:
- net +3V3 is gone; now on net +5V: J4.2
Changed lines of the file:
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@@
-    )
-  )
-  (symbol (lib_id "power:+3V3") (at 49.53 77.47 0) (unit 1)
-    (in_bom yes) (on_board yes) (dnp no)
-    (property "Reference" "#PWR032" (at 49.53 81.28 0)
-      (effects (font (size 1.27 1.27)) hide)
-    )
-    (property "Value" "+3V3" (at 49.53 73.7362 0)
-      (effects (font (size 1.27 1.27)))
-    )
-    (property "Footprint" "" (at 49.53 77.47 0)
-      (effects (font (size 1.27 1.27)) hide)
-    )
-    (property "Datasheet" "" (at 49.53 77.47 0)
-      (effects (font (size 1.27 1.27)) hide)
-    )
-    (pin "1")
-    (instances
-      (project "KAKAPO-20A"
-        (path "/e63e39d7-6ac0-4ffd-8aa3-1841a4541b55"
-          (reference "#PWR032") (unit 1)
-        )
-      )
     )
   )
@@
         )
       )
+    )
+  )
+  (symbol (lib_id "power:+5V") (at 49.53 77.47 0) (mirror y) (unit 1)
+    (in_bom yes) (on_board yes) (dnp no)
+    (property "Reference" "#PWR01" (at 49.53 81.28 0)
+      (effects (font (size 1.27 1.27)) hide)
+    )
+    (property "Value" "+5V" (at 49.53 73.66 0)
+      (effects (font (size 1.27 1.27)))
+    )
+    (property "Footprint" "" (at 49.53 77.47 0)
+      (effects (font (size 1.27 1.27)) hide)
+    )
+    (property "Datasheet" "" (at 49.53 77.47 0)
+      (effects (font (size 1.27 1.27)) hide)
+    )
+    (pin "1")
+    (instances
+      (project "KAKAPO-20A"
+        (path "/e63e39d7-6ac0-4ffd-8aa3-1841a4541b55"
+          (reference "#PWR01") (unit 1)
+        )
+      )
